Commit message: modified:   urdf/robott.urdf

File: urdf/robott.urdf (robot description, URDF)
Before this commit: robot qrobott, 1 links, 0 joints
Links:
- added link link1; visual mesh filename=package://robot_description/meshes/link1.stl scale=1.0 1.0 1.0
- added link link2; visual mesh filename=package://robot_description/meshes/link2.stl scale=1.0 1.0 1.0
- added link link_base; visual mesh filename=package://robot_description/meshes/link_base.stl scale=1.0 1.0 1.0
- link base_link: geometry visual box size=0 0 0
Joints:
- added joint base_link_to_link_base: type fixed, parent base_link, child link_base, origin xyz=0 0 0 rpy=0.0 0.0 0.0
- added joint link1_to_link2: type fixed, parent link1, child link2, origin xyz=0 0.0 0.0 rpy=-1.5 -1.5 0.0
- added joint link_base_to_link1: type fixed, parent link_base, child link1, origin xyz=0 0 0.24 rpy=0.0 0.0 0.0

Commit message: final assemble

File: urdf/robott.urdf (robot description, URDF)
Before this commit: robot qrobott, 4 links, 3 joints
Links:
- added link gripper_lite; visual mesh filename=package://robot_description/meshes/gripper_lite.stl scale=1.0 1.0 1.0
- added link link3; visual mesh filename=package://robot_description/meshes/link3.stl scale=1.0 1.0 1.0
- added link link4; visual mesh filename=package://robot_description/meshes/link4.stl scale=1.0 1.0 1.0
- added link link5; visual mesh filename=package://robot_description/meshes/link5.stl scale=1.0 1.0 1.0
- added link link6; visual mesh filename=package://robot_description/meshes/link6.stl scale=1.0 1.0 1.0
Joints:
- added joint link2_to_link3: type fixed, parent link2, child link3, origin xyz=0.2 0 0 rpy=3.14 0 1.57
- added joint link3_to_link4: type fixed, parent link3, child link4, origin xyz=0.09 -0.23 0 rpy=1.57 6.28 0
- added joint link4_to_link5: type fixed, parent link4, child link5, origin xyz=0 0 0 rpy=0 0 3.14
- added joint link5_to_link6: type fixed, parent link5, child link6, origin xyz=0 0 0.03 rpy=0 0 3.14
- added joint link6_to_gripper_lite: type fixed, parent link6, child gripper_lite, origin xyz=0 0 0.01 rpy=0 0 3.14
- joint link1_to_link2: origin xyz=0 0.0 0.0 rpy=-1.5 -1.5 0.0 -> xyz=0 0.0 0.0 rpy=-1.57 -1.57 0.0

Commit message: First build

File: urdf/robott.urdf (robot description, URDF)
Before this commit: robot qrobott, 9 links, 8 joints
Joints:
- joint link6_to_gripper_lite: axis (none) -> 0 0 1; limit (none) -> lower=-3.14 upper=3.14 effort=0 velocity=0; type fixed -> revolute

Commit message: added revolute joints

File: urdf/robott.urdf (robot description, URDF)
Before this commit: robot qrobott, 9 links, 8 joints
Joints:
- joint link1_to_link2: axis (none) -> 0 0 1; limit (none) -> lower=-3.14 upper=3.14 effort=0 velocity=0; type fixed -> revolute
- joint link2_to_link3: axis (none) -> 0 0 1; limit (none) -> lower=-3.14 upper=3.14 effort=0 velocity=0; type fixed -> revolute
- joint link3_to_link4: axis (none) -> 0 0 1; limit (none) -> lower=-3.14 upper=3.14 effort=0 velocity=0; type fixed -> revolute
- joint link4_to_link5: axis (none) -> 0 0 1; limit (none) -> lower=-3.14 upper=3.14 effort=0 velocity=0; type fixed -> revolute
- joint link5_to_link6: axis (none) -> 0 0 1; limit (none) -> lower=-3.14 upper=3.14 effort=0 velocity=0; type fixed -> revolute
- joint link_base_to_link1: axis (none) -> 0 0 1; limit (none) -> lower=-3.14 upper=3.14 effort=0 velocity=0; type fixed -> revolute

Commit message: added material and completed joints

File: urdf/robott.urdf (robot description, URDF)
Before this commit: robot qrobott, 9 links, 8 joints
Joints:
- joint link1_to_link2: limit lower=-3.14 upper=3.14 effort=0 velocity=0 -> lower=-1.31 upper=1.31 effort=0 velocity=0
- joint link2_to_link3: limit lower=-3.14 upper=3.14 effort=0 velocity=0 -> lower=-0.03 upper=2.62 effort=0 velocity=0
- joint link4_to_link5: axis 0 0 1 -> 0 1 0; limit lower=-3.14 upper=3.14 effort=0 velocity=0 -> lower=-1.08 upper=1.08 effort=0 velocity=0
